Commit message: sync 0.0.3-625-g35fca00a of https://www.lejuhub.com/highlydynamic/kuavo

File: models/biped_gen3.4/urdf/biped_v3.urdf (robot description, URDF)
Before this commit: robot biped_v3, 13 links, 12 joints
Links:
- link torso: mass 33.1207795 -> 31.4207795

File: models/biped_gen3.4/urdf/biped_v3_arm.urdf (robot description, URDF)
Before this commit: robot biped_v3, 15 links, 14 joints
Links:
- link l_hand_pitch: mass 0.6789 -> 0.774
- link r_hand_pitch: mass 0.6789 -> 0.774
