Commit message: sync 0.0.3-1352-g42de2e16 of https://www.lejuhub.com/highlydynamic/kuavo

File: models/biped_gen3.4/urdf/biped_v3_arm.urdf (robot description, URDF)
Before this commit: robot biped_v3, 15 links, 14 joints
Joints:
- joint l_arm_pitch: limit (none) -> lower=-3.14 upper=0.52 effort=20 velocity=1
- joint l_arm_roll: limit (none) -> lower=-0.35 upper=2.36 effort=20 velocity=1
- joint l_arm_yaw: limit (none) -> lower=-2.36 upper=2.36 effort=20 velocity=1
- joint l_forearm_pitch: limit (none) -> lower=-1.75 upper=1.75 effort=20 velocity=1
- joint l_forearm_yaw: limit (none) -> lower=-2.36 upper=2.36 effort=20 velocity=1
- joint l_hand_pitch: limit (none) -> lower=-0.26 upper=0.26 effort=20 velocity=1
- joint l_hand_roll: limit (none) -> lower=-0.17 upper=0.17 effort=20 velocity=1
- joint r_arm_pitch: limit (none) -> lower=-3.14 upper=3.14 effort=20 velocity=1
- joint r_arm_roll: limit (none) -> lower=-3.14 upper=3.14 effort=20 velocity=1
- joint r_arm_yaw: limit (none) -> lower=-3.14 upper=3.14 effort=20 velocity=1
- joint r_forearm_pitch: limit (none) -> lower=-3.14 upper=3.14 effort=20 velocity=1
- joint r_forearm_yaw: limit (none) -> lower=-3.14 upper=3.14 effort=20 velocity=1
- joint r_hand_pitch: limit (none) -> lower=-0.26 upper=0.26 effort=20 velocity=1
- joint r_hand_roll: limit (none) -> lower=-0.17 upper=0.17 effort=20 velocity=1
